Commit message: Upload my mods

File: p3dx_description/urdf/pioneer3dx.xacro (robot description, xacro)
@@ -25,16 +25,12 @@
 		<inertial>
 			<mass value="3.5" />
-			<!--<origin xyz="-0.025 0 -0.223"/> -->
 			<origin xyz="-0.05 0 0" />
 			<inertia ixx="1" ixy="0" ixz="0" iyy="1" iyz="0" izz="1" />
 		</inertial>
-		<visual name="base_visual">
+		<visual>
 			<origin xyz="-0.045 0 0.148" rpy="0 0 0" />
 			<geometry name="pioneer_geom">
 				<mesh filename="package://p3dx_description/meshes/chassis.stl" />
 			</geometry>
-			<material name="ChassisRed">
-				<color rgba="0.851 0.0 0.0 1.0" />
-			</material>
 		</visual>
 		<collision>
@@ -52,12 +48,9 @@
 			<inertia ixx="1" ixy="0" ixz="0" iyy="1" iyz="0" izz="1" />
 		</inertial>
-		<visual name="base_visual">
+		<visual>
 			<origin xyz="0 0 0" rpy="0 0 0" />
 			<geometry name="top_geom">
 				<mesh filename="package://p3dx_description/meshes/top.stl" />
 			</geometry>
-			<material name="TopBlack">
-				<color rgba="0.038 0.038 0.038 1.0" />
-			</material>
 		</visual>
 		<collision>
@@ -80,17 +73,14 @@
 			<inertia ixx="0.01" ixy="0" ixz="0" iyy="0.01" iyz="0" izz="0.01" />
 		</inertial>
-		<visual name="base_visual">
+		<visual>
 			<origin xyz="0 0 0" rpy="0 0 0" />
 			<geometry name="pioneer_geom">
 				<mesh filename="package://p3dx_description/meshes/swivel.stl" />
 			</geometry>
-			<material name="swivel">
-				<color rgba="0.5 0.5 0.5 1" />
-			</material>
-		</visual>
-		<collision>
-			<origin xyz="0 0 0" rpy="0 0 0" />
-			<geometry>
-				<box size="0 0 0" />
+		</visual>
+		<collision>
+			<origin xyz="0 0 0" rpy="0 0 0" />
+			<geometry>
+				<box size="0.01 0.01 0.01" />
 			</geometry>
 		</collision>
@@ -113,17 +103,14 @@
 				iyy="0.015218160428" iyz="-0.000004273467" izz="0.011763977943" />
 		</inertial>
-		<visual name="base_visual">
+		<visual>
 			<origin xyz="0 0 0" rpy="0 0 0" />
 			<geometry name="pioneer_geom">
 				<mesh filename="package://p3dx_description/meshes/center_hubcap.stl" />
 			</geometry>
-			<material name="swivel">
-				<color rgba="0.5 0.5 0.5 1" />
-			</material>
-		</visual>
-		<collision>
-			<origin xyz="0 0 0" rpy="0 0 0" />
-			<geometry>
-				<box size="0 0 0" />
+		</visual>
+		<collision>
+			<origin xyz="0 0 0" rpy="0 0 0" />
+			<geometry>
+				<box size="0.01 0.01 0.01" />
 			</geometry>
 		</collision>
@@ -146,12 +133,9 @@
 				iyy="0.015218160428" iyz="-0.000004273467" izz="0.011763977943" />
 		</inertial>
-		<visual name="base_visual">
+		<visual>
 			<origin xyz="0 0 0" rpy="0 0 0" />
 			<geometry name="pioneer_geom">
 				<mesh filename="package://p3dx_description/meshes/center_wheel.stl" />
 			</geometry>
-			<material name="WheelBlack">
-				<color rgba="0.117 0.117 0.117 1" />
-			</material>
 		</visual>
 		<collision>
@@ -176,17 +160,14 @@
 			<inertia ixx="1" ixy="0" ixz="0" iyy="1" iyz="0" izz="1" />
 		</inertial>
-		<visual name="front_sonar_vis">
+		<visual>
 			<origin rpy="0 0 0" xyz="0 0 0" />
 			<geometry name="pioneer_geom">
 				<mesh filename="package://p3dx_description/meshes/front_sonar.stl" />
 			</geometry>
-			<material name="SonarYellow">
-				<color rgba="0.715 0.583 0.210 1.0" />
-			</material>
 		</visual>
 		<collision>
 			<origin rpy="0 0 0" xyz="0 0 0" />
 			<geometry>
-				<box size="0 0 0" />
+				<box size="0.01 0.01 0.01" />
 			</geometry>
 		</collision>
@@ -200,5 +181,5 @@
 	<link name="lms100">
 		<inertial>
-			<mass value="1e-5" />
+			<mass value="0.16" />
 			<origin xyz="0 0 0" rpy="0 0 0" />
 			<inertia ixx="1e-6" ixy="0" ixz="0" iyy="1e-6" iyz="0" izz="1e-6" />
@@ -219,7 +200,34 @@
 	<joint name="lms100_joint" type="fixed">
 		<axis xyz="0 1 0" />
-		<origin xyz="0.16 0 0.15" rpy="0 0 0" />
+		<origin xyz="0.10 0 0.272" rpy="0 0 0" />
 		<parent link="base_link" />
 		<child link="lms100" />
 	</joint>
+	<!-- Camera -->
+	<link name="camera_link">
+	  <collision>
+		    <origin xyz="0 0 0" rpy="0 0 0"/>
+		    <geometry>
+		  	<box size="0.05 0.05 0.05"/>
+		    </geometry>
+	  </collision>
+	  <visual>
+		    <origin xyz="0 0 0" rpy="0 0 0"/>
+		    <geometry>
+		 	<box size="0.05 0.05 0.05"/>
+		    </geometry>
+		    <material name="red"/>
+	  </visual>
+	  <inertial>
+		    <mass value="1e-5" />
+		    <origin xyz="0 0 0" rpy="0 0 0"/>
+		    <inertia ixx="1e-6" ixy="0" ixz="0" iyy="1e-6" iyz="0" izz="1e-6" />
+	  </inertial>
+	</link>
+	<joint name="camera_joint" type="fixed">
+	  <axis xyz="0 1 0" />
+	  <origin xyz="0 0 1" rpy="0 0 0"/>
+	  <parent link="base_link"/>
+	  <child link="camera_link"/>
+	</joint>
 </robot>

File: p3dx_description/urdf/pioneer3dx_wheel.xacro (robot description, xacro)
@@ -29,5 +29,5 @@
 					iyz="0" izz="0.011763977943" />
 			</inertial>
-			<visual name="base_visual">
+			<visual>
 				<origin xyz="0 0 0" rpy="0 0 0" />
 				<geometry name="pioneer_geom">
@@ -59,5 +59,5 @@
 					iyz="0" izz="0.011763977943" />
 			</inertial>
-			<visual name="base_visual">
+			<visual>
 				<origin xyz="0 0 0" rpy="0 0 0" />
 				<geometry name="pioneer_geom">
@@ -71,5 +71,5 @@
 				<origin xyz="0 0 0" rpy="0 0 0" />
 				<geometry>
-					<box size="0 0 0" />
+					<box size="0.01 0.01 0.01" />
 				</geometry>
 			</collision>
